File: can_interface.kicad_sch (KiCad schematic)
At the start: 3 parts, among them U11 MCP2562-E-SN

Commit message: Update Including Revisions 1.1 and 2
Parts:
- added C30: C100n, Capacitor_SMD:C_0805_2012Metric_Pad1.18x1.45mm_HandSolder, symbol Device:C
- added C36, C39: C22p, Capacitor_SMD:C_0805_2012Metric_Pad1.18x1.45mm_HandSolder, symbol Device:C
- added R3, R6: R0, Resistor_SMD:R_0805_2012Metric_Pad1.20x1.40mm_HandSolder, symbol Device:R
- added U10: MCP2518FDT-E/SL, MCP2518FDT-E-SL:SOIC14_SL_MCH, symbol 2024-05-05_05-04-59:MCP2518FDT-E_SL
- added Y1: Crystal_GND24_Small, Crystal:Crystal_SMD_Abracon_ABM3C-4Pin_5.0x3.2mm, symbol Device:Crystal_GND24_Small
Connections:
- net GND: now also C30.2, C36.1, C39.1, U10.7 (VSS), Y1.2, Y1.4
- net IOREF: now also C30.1, U10.14 (VDD)
- net canrx: now also R6.1, U10.2 (RXCAN)
- net cantx: now also R3.2, U10.1 (TXCAN)
- net can_h+ renamed can+
- net can_l- renamed can-
- new net: C39.2, U10.6 (OSC1), Y1.3
- new net: C36.2, U10.5 (OSC2), Y1.1
- new net cipo-cantx: R3.1, U10.12 (SDO)
- new net copi: U10.11 (SDI)
- new net cs-canrx: R6.2, U10.13 (nCS)
- new net int: U10.4 (*INT)
- new net sck: U10.10 (SCK)
- no-connect marks 0 -> 3
Other:
- moved on the sheet: C32, C33, U11
