File: Pico_LCC.kicad_sch (KiCad schematic)
At the start: 20 parts, among them J1 Screw_Terminal_01x12, J2 RJHSE508002, J3 SM04B-SRSS-TB, J4 SM04B-SRSS-TB, U1 Pico, U14 SN3257QPWRQ1

Commit message: Update Including Revisions 1.1 and 2
Parts:
- removed J4: SM04B-SRSS-TB, SM04B_SRSS_TB:CONN_SM04B-SRSS-TB_JST, symbol SM04B_SRSS_TB:SM04B-SRSS-TB
- removed R3, R6: R2.2k, Resistor_SMD:R_0805_2012Metric_Pad1.20x1.40mm_HandSolder, symbol Device:R
- added JP6: SolderJumper_2_Open, Jumper:SolderJumper-2_P1.3mm_Open_RoundedPad1.0x1.5mm, symbol Jumper:SolderJumper_2_Open
- added R17: R120, Resistor_SMD:R_0805_2012Metric_Pad1.20x1.40mm_HandSolder, symbol Device:R
- JP1: footprint Jumper:SolderJumper-2_P1.3mm_Open_RoundedPad1.0x1.5mm -> Jumper:SolderJumper-2_P1.3mm_Bridged_RoundedPad1.0x1.5mm; symbol Jumper:SolderJumper_2_Open -> Jumper:SolderJumper_2_Bridged
Connections:
- net dcc_p: now also JP6.1 (A); no longer U1.34 (GPIO28_ADC2)
- net can_h+ renamed can+
- net can+: now also R17.2
- net can_l- renamed can-
- net can-: now also R17.1
- net canrx renamed spi0_cs
- net cantx renamed spi0_rx
- net i2c1_scl renamed spi0_tx
- net i2c1_sda renamed spi0_sck
- new net spi0_int: JP6.2 (B), U1.34 (GPIO28_ADC2)
Other:
- sheet CAN Interface ports: added can+, can-, cipo-cantx, copi, cs-canrx, int, sck; removed can_h+, can_l-, canrx, cantx
- moved on the sheet: C29, J2A, J2B, U14

Commit message: v4
Parts:
- removed U1: Pico, RPi_Pico:RPi_Pico_SMD_TH, symbol MCU_RaspberryPi_and_Boards:Pico
- added A1: RaspberryPi_Pico, Module:RaspberryPi_Pico_Common_SMD, symbol MCU_Module:RaspberryPi_Pico
- added C2, C3: C100n, Capacitor_SMD:C_0805_2012Metric_Pad1.18x1.45mm_HandSolder, symbol Device:C
- added J4: SM04B-SRSS-TB, SM04B_SRSS_TB:CONN_SM04B-SRSS-TB_JST, symbol SM04B_SRSS_TB:SM04B-SRSS-TB
- added R4, R5: R2.2k, Resistor_SMD:R_0805_2012Metric_Pad1.20x1.40mm_HandSolder, symbol Device:R
- added U2: MCP2562-E-SN, Package_SO:SOIC-8_3.9x4.9mm_P1.27mm, symbol Interface_CAN_LIN:MCP2562-E-SN
- renumbered C29 to C1, JP2 to JP1, JP3 to JP2, JP4 to JP3, JP5 to JP4, JP1 to JP5, R17 to R1, R9 to R2, R12 to R3, U14 to U1
Connections:
- net spi0_int is gone; now on net +3.3V: JP6.2 (B)
- net +3.3V: now also A1.36 (3V3), C2.1, J4.2, R4.1, R5.1, U2.5 (Vio)
- net +5V: now also A1.40 (VBUS), C3.1, U2.3 (VDD)
- net GND: now also A1.13 (GND), A1.18 (GND), A1.23 (GND), A1.28 (GND), A1.3 (GND), A1.33 (AGND), A1.38 (GND), A1.8 (GND), C2.2, C3.2, J4.1, U2.2 (VSS), U2.8 (STBY)
- net adc0: now also A1.31 (GPIO26_ADC0)
- net adc1: now also A1.32 (GPIO27_ADC1)
- net adc_sel: now also A1.29 (GPIO22)
- net can+: now also U2.7 (CANH)
- net can-: now also U2.6 (CANL)
- net dcc_en_A: now also A1.2 (GPIO1)
- net dcc_en_B: now also A1.7 (GPIO5)
- net dcc_en_C: now also A1.12 (GPIO9)
- net dcc_en_D: now also A1.17 (GPIO13)
- net dcc_p: now also A1.34 (GPIO28_ADC2); no longer JP6.1 (A)
- net dir_A: now also A1.4 (GPIO2)
- net dir_B: now also A1.9 (GPIO6)
- net dir_C: now also A1.14 (GPIO10)
- net dir_D: now also A1.19 (GPIO14)
- net i2c0_scl: now also A1.27 (GPIO21)
- net i2c0_sda: now also A1.26 (GPIO20)
- net nFault_A: now also A1.1 (GPIO0)
- net nFault_B: now also A1.6 (GPIO4)
- net nFault_C: now also A1.11 (GPIO8)
- net nFault_D: now also A1.16 (GPIO12)
- net pwm_A: now also A1.5 (GPIO3)
- net pwm_B: now also A1.10 (GPIO7)
- net pwm_C: now also A1.15 (GPIO11)
- net pwm_D: now also A1.20 (GPIO15)
- new net: A1.35 (ADC_VREF), JP6.1 (A)
- new net canrx: A1.22 (GPIO17), U2.4 (RXD)
- new net cantx: A1.21 (GPIO16), U2.1 (TXD)
- new net i2c1_scl: A1.25 (GPIO19), J4.4, R4.2
- new net i2c1_sda: A1.24 (GPIO18), J4.3, R5.2
- no-connect marks 9 -> 5
Other:
- removed sheet CAN Interface
- moved on the sheet: C1, H1, H2, H3, H4, J1, J2A, J2B, J3, JP1, JP2, JP3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
