File: block_driver.kicad_sch (KiCad schematic)
At the start: 11 parts, among them U4 SN74HC253DR, U5 DRV8874PWPR

Commit message: v4
Parts:
- renumbered C14 to C10, C8 to C4, C9 to C5, C10 to C6, C11 to C7, C12 to C8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
Other:
- moved on the sheet: C10, C4, C5, C6, C7, C8, C9, R6, R7, U4, U5
