File: dcc_isolator.kicad_sch (KiCad schematic)
At the start: 8 parts, among them U12 6N137, U13 6N137

Commit message: v4
Parts:
- renumbered C34 to C32, C35 to C33, R13 to R14, R14 to R15, R15 to R16, R16 to R17
Other:
- moved on the sheet: C32, C33, R14, R15, R16, R17, U12, U13
