File: Pico_LCC.kicad_pcb (KiCad board)
At the start: 2 copper layers, 85 x 100 mm, 75 parts, among them J1 Screw_Terminal_01x12, J2 RJHSE508002, J3 SM04B-SRSS-TB, J4 SM04B-SRSS-TB, U1 Pico, U11 MCP2562-E-SN, U12 6N137, U13 6N137, U14 SN3257QPWRQ1, U2 SN74HC253DR, U3 DRV8874PWPR, U4 SN74HC253DR, U5 DRV8874PWPR, U6 SN74HC253DR, U7 DRV8874PWPR, U8 SN74HC253DR, U9 DRV8874PWPR

Commit message: Update Including Revisions 1.1 and 2
Parts:
- removed J4: SM04B-SRSS-TB, SM04B_SRSS_TB:CONN_SM04B-SRSS-TB_JST
- added C30: C100n, Capacitor_SMD:C_0805_2012Metric_Pad1.18x1.45mm_HandSolder, F.Cu at (82.0, 83.2)
- added C36: C22p, Capacitor_SMD:C_0805_2012Metric_Pad1.18x1.45mm_HandSolder, F.Cu at (88.4, 98.0)
- added C39: C22p, Capacitor_SMD:C_0805_2012Metric_Pad1.18x1.45mm_HandSolder, F.Cu at (93.4, 94.6)
- added JP6: SolderJumper_2_Open, Jumper:SolderJumper-2_P1.3mm_Open_RoundedPad1.0x1.5mm, F.Cu at (76.6, 81.6)
- added R17: R120, Resistor_SMD:R_0805_2012Metric_Pad1.20x1.40mm_HandSolder, F.Cu at (91.8, 102.2)
- added U10: MCP2518FDT-E/SL, MCP2518FDT-E-SL:SOIC14_SL_MCH, F.Cu at (87.2, 88.1)
- added Y1: Crystal_GND24_Small, Crystal:Crystal_SMD_Abracon_ABM3C-4Pin_5.0x3.2mm, F.Cu at (89.2, 94.6)
- JP1: footprint Jumper:SolderJumper-2_P1.3mm_Open_RoundedPad1.0x1.5mm -> Jumper:SolderJumper-2_P1.3mm_Bridged_RoundedPad1.0x1.5mm
- R3, R6: value R2.2k -> R0
- moved R3 33.8 mm to (82.2, 93.8), turned to 0 degrees
- moved R6 33.6 mm to (83.4, 97.0), turned to 180 degrees
- moved JP1 14.7 mm to (105.8, 110.8)
- moved C29 8.05 mm to (87.1, 106.3)
- moved C33 8.05 mm to (80.8, 102.2)
- moved U11 8.05 mm to (85.8, 102.2)
Connections:
- net /can_h+ renamed /can+
- net /can_l- renamed /can-
- R3 pad 1: +3.3V -> /spi0_rx
- R3 pad 2: /i2c1_scl -> /CAN Interface/cantx
- R6 pad 1: +3.3V -> /CAN Interface/canrx
- R6 pad 2: /i2c1_sda -> /spi0_cs
- U1 pad 21: /cantx -> /spi0_rx
- U1 pad 22: /canrx -> /spi0_cs
- U1 pad 24: /i2c1_sda -> /spi0_sck
- U1 pad 25: /i2c1_scl -> /spi0_tx
- U1 pad 34: /dcc_p -> /spi0_int
- U11 pad 1: /cantx -> /CAN Interface/cantx
- U11 pad 4: /canrx -> /CAN Interface/canrx
Routing:
- net /spi0_int: track 0.00 -> 61.6 mm, vias 0 -> 2
- net /spi0_cs: track 0.00 -> 32.9 mm
- net /spi0_tx: track 0.00 -> 32.2 mm
- net /dcc_p: track 159.3 -> 130.2 mm, vias 6 -> 7
- net /canrx: track 28.0 -> 0.00 mm
- net GND: track 165.5 -> 140.1 mm, vias 82 -> 84
- net +3.3V: track 390.9 -> 415.8 mm, vias 23 -> 25
- net /spi0_rx: track 0.00 -> 23.0 mm
- net /spi0_sck: track 0.00 -> 20.9 mm
- net /cantx: track 20.6 -> 0.00 mm
- net /i2c1_scl: track 17.4 -> 0.00 mm
- net /i2c1_sda: track 16.8 -> 0.00 mm
- net /CAN Interface/canrx: track 0.00 -> 15.1 mm
- net /CAN Interface/cantx: track 0.00 -> 9.52 mm
- net /can_shield: track 26.2 -> 34.7 mm
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Other:
- board text added: "A+"
- board text added: "A-"
- board text added: "B+"
- board text added: "B-"
- board text added: "C+"
- board text added: "C-"
- board text added: "CAN Term"
- board text added: "D+"
- board text added: "D-"
- board text added: "DCC+"
- board text added: "DCC-"
- board text added: "GND"
- board text added: "LCC JACK"
- board text added: "Pico LCC v2"
- board text added: "QWIIC 0"
- board text added: "VTRACK"
- board text removed: "Pico LCC v1"

Commit message: v4
Parts:
- removed the C30 at (82.0, 83.2)
- removed the C32 at (94.7, 44.8)
- removed the C33 at (80.8, 102.2)
- removed C36, C39: C22p, Capacitor_SMD:C_0805_2012Metric_Pad1.18x1.45mm_HandSolder
- removed the R3 at (82.2, 93.8)
- removed the R6 at (83.4, 97.0)
- removed the U1 at (79.2, 51.0)
- removed the U10 at (87.2, 88.1)
- removed the U11 at (85.8, 102.2)
- removed Y1: Crystal_GND24_Small, Crystal:Crystal_SMD_Abracon_ABM3C-4Pin_5.0x3.2mm
- added A1: RaspberryPi_Pico, Module:RaspberryPi_Pico_Common_SMD, F.Cu at (79.2, 51.0)
- added C2: C100n, Capacitor_SMD:C_0805_2012Metric_Pad1.18x1.45mm_HandSolder, F.Cu at (94.6, 44.7)
- added C3: C100n, Capacitor_SMD:C_0805_2012Metric_Pad1.18x1.45mm_HandSolder, F.Cu at (80.8, 102.2)
- added J4: SM04B-SRSS-TB, SM04B_SRSS_TB:CONN_SM04B-SRSS-TB_JST, F.Cu at (106.8, 69.0)
- added R4: R2.2k, Resistor_SMD:R_0805_2012Metric_Pad1.20x1.40mm_HandSolder, F.Cu at (101.5, 66.0)
- added R5: R2.2k, Resistor_SMD:R_0805_2012Metric_Pad1.20x1.40mm_HandSolder, F.Cu at (98.5, 67.1)
- added U2: MCP2562-E-SN, Package_SO:SOIC-8_3.9x4.9mm_P1.27mm, F.Cu at (85.8, 102.2)
- moved JP6 45.5 mm to (94.6, 39.9)
- renumbered C29 to C1, C7 to C10, C8 to C11, C9 to C12, C10 to C13, C11 to C14, C12 to C15, C13 to C16, C14 to C17, C15 to C18, C16 to C19, C17 to C20, C18 to C21, C19 to C22, C20 to C23, C21 to C24, C22 to C25, C23 to C26, C24 to C27, C25 to C28, C26 to C29, C27 to C30, C28 to C31, C34 to C32, C35 to C33, C1 to C4, C2 to C5, C3 to C6, C4 to C7, C5 to C8, C6 to C9, JP2 to JP1, JP3 to JP2, JP4 to JP3, JP5 to JP4, JP1 to JP5, R17 to R1, R7 to R10, R8 to R11, R10 to R12, R11 to R13, R13 to R14, R14 to R15, R15 to R16, R16 to R17, R9 to R2, R12 to R3, R1 to R6, R2 to R7, R4 to R8, R5 to R9, U14 to U1, U8 to U10, U9 to U11, U2 to U4, U3 to U5, U4 to U6, U5 to U7, U6 to U8, U7 to U9
Connections:
- JP6 pad 1: /dcc_p -> Net-(A1-ADC_VREF)
- JP6 pad 2: /spi0_int -> +3.3V
Routing:
- net /spi0_int: track 61.6 -> 0.00 mm, vias 2 -> 0
- net /dcc_p: track 130.2 -> 179.4 mm
- net /canrx: track 0.00 -> 39.2 mm
- net /spi0_cs: track 32.9 -> 0.00 mm
- net /spi0_tx: track 32.2 -> 0.00 mm
- net /cantx: track 0.00 -> 32.0 mm
- net /spi0_rx: track 23.0 -> 0.00 mm
- net /spi0_sck: track 20.9 -> 0.00 mm
- net /i2c1_scl: track 0.00 -> 17.7 mm
- net /i2c1_sda: track 0.00 -> 16.9 mm
- net /CAN Interface/canrx: track 15.1 -> 0.00 mm
- net +5V: track 172.2 -> 184.1 mm, vias 3 -> 5
- net /CAN Interface/cantx: track 9.52 -> 0.00 mm
- net GND: track 140.1 -> 148.6 mm, vias 84 -> 97
- net Net-(U10-OSC1): track 8.02 -> 0.00 mm
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Other:
- board text added: "Pico LCC Booster"
- board text added: "QWIIC 1"
- board text added: "Rev ${REVISION}"
- board text removed: "Pico LCC v2"

Commit message: v4 with Stencil and Frame
Parts:
- moved JP5 29.2 mm to (130.8, 125.8)
- moved C17 29.2 mm to (65.3, 75.1)
- moved C24 29.2 mm to (65.3, 91.9)
- moved C31 29.2 mm to (65.3, 108.6)
- moved C6 29.2 mm to (67.7, 69.4)
- moved A1 29.2 mm to (104.2, 66.0)
- moved C1 29.2 mm to (112.1, 121.3)
- moved C10 29.2 mm to (65.4, 58.4)
- moved C11 29.2 mm to (70.9, 82.1)
- moved C12 29.2 mm to (81.4, 75.6)
- moved C14 29.2 mm to (69.4, 88.4)
- moved C15 29.2 mm to (63.4, 87.1)
- moved C16 29.2 mm to (71.6, 86.1)
- moved C18 29.2 mm to (70.9, 98.9)
- moved C19 29.2 mm to (81.4, 92.4)
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